File: IoT.kicad_pcb (KiCad board)
At the start: 2 copper layers, 48.3 x 31.6 mm, 56 parts, among them J1 Conn_Coaxial, J2 Conn_01x05, J3 BAT, U1 STM32WLE5C8Ux, U2 BMP280, U3 SHT4x, U5 INA180A1, U6 TPS62177DQC, Y1 32.768kHz, Y2 32MHz

Commit message: Add files via upload
Parts:
- moved J1 0.10 mm to (118.0, 91.1)
Routing:
- net Net-(J1-In): track 6.96 -> 8.38 mm
Changed lines of the file:
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@@
   )
   (footprint "Connector_Coaxial:SMA_Samtec_SMA-J-P-X-ST-EM1_EdgeMount" (layer "F.Cu")
-    (at 117.96 91.005 -90)
+    (at 117.975 91.1 -90)
     (descr "Connector SMA, 0Hz to 20GHz, 50Ohm, Edge Mount (http://suddendocs.samtec.com/prints/sma-j-p-x-st-em1-mkt.pdf)")
     (tags "SMA Straight Samtec Edge Mount")
@@
   (segment (start 148.8 91.25) (end 151.1552 88.8948) (width 0.2) (layer "F.Cu") (net 5))
   (segment (start 151.1552 88.8948) (end 151.156 88.8948) (width 0.2) (layer "F.Cu") (net 5))
-  (segment (start 143.8678 89.392) (end 143.8678 91.2716) (width 0.25) (layer "F.Cu") (net 6))
-  (segment (start 141.9628 89.3942) (end 143.8656 89.3942) (width 0.25) (layer "F.Cu") (net 6))
+  (segment (start 141.9461 89.3775) (end 141.9628 89.3942) (width 0.35) (layer "F.Cu") (net 6))
+  (segment (start 140.3525 89.4) (end 140.375 89.3775) (width 0.35) (layer "F.Cu") (net 6))
   (segment (start 140.3917 89.3942) (end 140.375 89.3775) (width 0.2) (layer "F.Cu") (net 6))
+  (segment (start 141.9628 89.3942) (end 143.8656 89.3942) (width 0.35) (layer "F.Cu") (net 6))
   (segment (start 141.9628 89.3942) (end 141.9503 89.3817) (width 0.2) (layer "F.Cu") (net 6))
-  (segment (start 141.9628 89.3942) (end 140.3917 89.3942) (width 0.2) (layer "F.Cu") (net 6))
-  (segment (start 143.8656 89.3942) (end 143.8678 89.392) (width 0.25) (layer "F.Cu") (net 6))
-  (segment (start 138.8 89.4) (end 140.3525 89.4) (width 0.2) (layer "F.Cu") (net 6))
-  (segment (start 140.3525 89.4) (end 140.375 89.3775) (width 0.2) (layer "F.Cu") (net 6))
+  (segment (start 143.8656 89.3942) (end 143.8678 89.392) (width 0.35) (layer "F.Cu") (net 6))
+  (segment (start 143.8678 91.2716) (end 143.8678 89.392) (width 0.35) (layer "F.Cu") (net 6))
+  (segment (start 138.8 89.4) (end 140.3525 89.4) (width 0.35) (layer "F.Cu") (net 6))
+  (segment (start 140.375 89.3775) (end 141.9461 89.3775) (width 0.35) (layer "F.Cu") (net 6))
   (segment (start 148.8 88.1705) (end 148.7932 88.1705) (width 0.2) (layer "F.Cu") (net 7))
   (segment (start 149.656 87.3145) (end 148.8 88.1705) (width 0.2) (layer "F.Cu") (net 7))
@@
   (segment (start 145.5928 89.392) (end 147.5717 89.392) (width 0.2) (layer "F.Cu") (net 7))
   (segment (start 149.656 83.3795) (end 149.656 87.3145) (width 0.2) (layer "F.Cu") (net 7))
-  (segment (start 138.85 91.175) (end 139.5025 90.5225) (width 0.2) (layer "F.Cu") (net 8))
-  (segment (start 136.4878 91.1237) (end 138.2753 91.1237) (width 0.25) (layer "F.Cu") (net 8))
-  (segment (start 139.5025 90.5225) (end 140.375 90.5225) (width 0.2) (layer "F.Cu") (net 8))
-  (segment (start 138.8 92.9792) (end 138.8 91.125) (width 0.2) (layer "F.Cu") (net 8))
-  (segment (start 138.2753 91.1237) (end 138.2798 91.1192) (width 0.25) (layer "F.Cu") (net 8))
+  (segment (start 138.8 91.125) (end 139.7725 91.125) (width 0.35) (layer "F.Cu") (net 8))
   (segment (start 138.8 91.125) (end 138.85 91.175) (width 0.2) (layer "F.Cu") (net 8))
-  (segment (start 133.0198 91.1237) (end 134.7378 91.1237) (width 0.25) (layer "F.Cu") (net 9))
-  (segment (start 127.7858 91.1237) (end 129.5123 91.1237) (width 0.25) (layer "F.Cu") (net 10))
+  (segment (start 139.7725 91.125) (end 140.375 90.5225) (width 0.35) (layer "F.Cu") (net 8))
+  (segment (start 138.8 91.125) (end 138.75 91.075) (width 0.35) (layer "F.Cu") (net 8))
+  (segment (start 138.8 91.125) (end 138.8 92.9792) (width 0.35) (layer "F.Cu") (net 8))
+  (segment (start 136.75 91.075) (end 138.75 91.075) (width 0.35) (layer "F.Cu") (net 8))
+  (segment (start 132.85 91.1) (end 134.675 91.1) (width 0.35) (layer "F.Cu") (net 9))
+  (segment (start 134.675 91.1) (end 134.7 91.075) (width 0.35) (layer "F.Cu") (net 9))
+  (segment (start 127.7858 91.1237) (end 129.5123 91.1237) (width 0.35) (layer "F.Cu") (net 10))
   (segment (start 131.2903 91.1192) (end 131.2948 91.1237) (width 0.25) (layer "F.Cu") (net 10))
-  (segment (start 129.5168 91.1192) (end 131.2903 91.1192) (width 0.25) (layer "F.Cu") (net 10))
-  (segment (start 129.5123 91.1237) (end 129.5168 91.1192) (width 0.25) (layer "F.Cu") (net 10))
+  (segment (start 131.125 91.1) (end 129.536 91.1) (width 0.35) (layer "F.Cu") (net 10))
+  (segment (start 129.5123 91.1237) (end 129.5168 91.1192) (width 0.35) (layer "F.Cu") (net 10))
+  (segment (start 127.7903 91.1192) (end 127.7858 91.1237) (width 0.25) (layer "F.Cu") (net 10))
+  (segment (start 129.536 91.1) (end 129.5168 91.1192) (width 0.35) (layer "F.Cu") (net 10))
   (segment (start 129.4593 91.1237) (end 129.5168 91.0662) (width 0.25) (layer "F.Cu") (net 10))
   (segment (start 147.2272 93.0076) (end 147.193 92.9734) (width 0.25) (layer "F.Cu") (net 11))
@@
   (segment (start 121.835 71.45) (end 134.395 71.45) (width 0.2) (layer "F.Cu") (net 20))
   (segment (start 120.405 66.03) (end 122.778896 66.03) (width 0.2) (layer "F.Cu") (net 20))
-  (segment (start 119.0044 91.1192) (end 125.9608 91.1192) (width 0.25) (layer "F.Cu") (net 21))
+  (segment (start 117.775 91.1) (end 125.9371 91.1) (width 0.35) (layer "F.Cu") (net 21))
+  (segment (start 125.9371 91.1) (end 125.9608 91.1237) (width 0.35) (layer "F.Cu") (net 21))
+  (segment (start 126 91.05) (end 125.955 91.005) (width 0.25) (layer "F.Cu") (net 21))
+  (segment (start 125.9608 91.0892) (end 126 91.05) (width 0.25) (layer "F.Cu") (net 21))
+  (segment (start 117.7987 91.1237) (end 117.775 91.1) (width 0.25) (layer "F.Cu") (net 21))
+  (segment (start 125.9608 91.1237) (end 125.9608 91.0892) (width 0.25) (layer "F.Cu") (net 21))
   (segment (start 154.217127 77.449227) (end 153.9579 77.19) (width 0.25) (layer "F.Cu") (net 22))
   (segment (start 153.9579 77.19) (end 152.3455 77.19) (width 0.25) (layer "F.Cu") (net 22))
@@
   (segment (start 138.4815 85.1415) (end 138.43 85.09) (width 0.25) (layer "B.Cu") (net 43))
   (segment (start 140.97 85.1415) (end 138.4815 85.1415) (width 0.25) (layer "B.Cu") (net 43))
+  (zone (net 0) (net_name "") (layer "B.Cu") (hatch edge 0.5)
+    (connect_pads (clearance 0))
+    (min_thickness 0.25) (filled_areas_thickness no)
+    (keepout (tracks not_allowed) (vias not_allowed) (pads not_allowed) (copperpour not_allowed) (footprints allowed))
+    (fill (thermal_gap 0.5) (thermal_bridge_width 0.5))
+    (polygon
+      (pts
+        (xy 115.475 85.925)
+        (xy 145.05 85.95)
+        (xy 145.05 86.675)
+        (xy 115.475 86.7)
+      )
+    )
+  )
   (zone (net 0) (net_name "") (layer "B.Cu") (name "abc") (hatch edge 0.5)
     (connect_pads yes (clearance 0))
@@
       )
     )
+  )
+  (zone (net 0) (net_name "") (layer "B.Cu") (hatch edge 0.5)
+    (connect_pads (clearance 0))
+    (min_thickness 0.25) (filled_areas_thickness no)
+    (keepout (tracks not_allowed) (vias not_allowed) (pads not_allowed) (copperpour not_allowed) (footprints allowed))
+    (fill (thermal_gap 0.5) (thermal_bridge_width 0.5))
+    (polygon
+      (pts
+        (xy 152.05 84.125)
+        (xy 153.075 84.125)
+        (xy 153.2 95.275)
+        (xy 152.175 95.275)
+      )
+    )
