File: IoT.kicad_sch (KiCad schematic)
At the start: 56 parts, among them J1 Conn_Coaxial, J2 Conn_01x05, J3 BAT, U1 STM32WLE5C8Ux, U2 BMP280, U3 SHT4x, U5 INA180A1, U6 TPS62177DQC, Y1 32.768kHz, Y2 32MHz

Commit message: Add files via upload
Other:
- note added: "3.3V"
